Commit message: feat: complete NBV autonomous exploration stack with sensor fusion and Nav2
Full implementation of:
- NBV planning library (OccupancyMapper, OutlineExtractor, CandidateGenerator, NBVScorer)
- Multi-sensor fusion node (LiDAR + Radar + RGB-D → /fused_scan)
- EKF localization (robot_localization + Madgwick IMU filter)
- SLAM Toolbox mapping with Nav2 navigation stack
- 4WD Mecanum robot URDF with Ignition Gazebo 6 simulation
- Modular launch system with startup sequencing (T+0/12/17/22 s)
- Cleaned codebase: consistent naming, dead code removed, no duplication

File: src/my_awesome_robot/urdf/robot.urdf.xacro (robot description, xacro)
@@ -1,198 +1,755 @@
 <?xml version="1.0"?>
-<robot name="my_awesome_robot" xmlns:xacro="http://www.ros.org/wiki/xacro">
-  <!-- ===================== -->
-  <!-- Parameters            -->
-  <!-- ===================== -->
-  <!-- Camera -->
-  <xacro:property name="cameraSize" value="0.05"/>
-  <xacro:property name="cameraMass" value="0.1"/>
-  <!-- Wheels -->
-  <xacro:property name="wheel_radius" value="0.1"/>
-  <xacro:property name="wheel_width"  value="0.05"/>
-  <xacro:property name="wheel_x" value="0.1"/>
-  <xacro:property name="wheel_y" value="0.15"/>
-  <!-- Chassis -->
-  <xacro:property name="chassis_x" value="0.4"/>
-  <xacro:property name="chassis_y" value="0.2"/>
-  <xacro:property name="chassis_z" value="0.1"/>
-  <!-- Xacro supports $(find pkg); $(find-pkg-share ...) is NOT a xacro command -->
-  <xacro:include filename="$(find my_awesome_robot)/urdf/robot.gazebo"/>
-  <!-- Materials -->
-  <material name="white"><color rgba="1 1 1 1"/></material>
-  <material name="green"><color rgba="0 0.9 0.2 1"/></material>
-  <material name="gray"><color rgba="0.4 0.4 0.4 1"/></material>
-  <!-- ===================== -->
-  <!-- Frames / Links         -->
-  <!-- ===================== -->
-  <!-- Root link without inertia -->
-  <link name="base_link"/>
-  <!-- Chassis -->
-  <joint name="chassis_joint" type="fixed">
+<robot name="autonomous_mobile_robot" xmlns:xacro="http://ros.org/wiki/xacro">
+  <!-- ================================================================ -->
+  <!-- XACRO PROPERTIES (tune geometry in one place)                     -->
+  <!-- ================================================================ -->
+  <xacro:property name="chassis_length"  value="0.50"/>
+  <xacro:property name="chassis_width"   value="0.30"/>
+  <xacro:property name="chassis_height"  value="0.08"/>
+  <xacro:property name="chassis_mass"    value="3.0"/>
+  <xacro:property name="upper_deck_length" value="0.38"/>
+  <xacro:property name="upper_deck_width"  value="0.26"/>
+  <xacro:property name="upper_deck_height" value="0.005"/>
+  <xacro:property name="upper_deck_mass"   value="0.3"/>
+  <xacro:property name="wheel_radius"    value="0.10"/>
+  <xacro:property name="wheel_width"     value="0.06"/>
+  <xacro:property name="wheel_mass"      value="0.4"/>
+  <xacro:property name="wheel_sep"       value="0.34"/>   <!-- center-to-center Y -->
+  <xacro:property name="wheelbase"       value="0.30"/>   <!-- front-to-rear X -->
+  <!-- ================================================================ -->
+  <!-- XACRO MACROS                                                      -->
+  <!-- ================================================================ -->
+  <!-- Box inertia macro -->
+  <xacro:macro name="box_inertia" params="m x y z">
+    <inertial>
+      <mass value="${m}"/>
+      <inertia ixx="${m/12.0*(y*y+z*z)}" ixy="0" ixz="0"
+               iyy="${m/12.0*(x*x+z*z)}" iyz="0"
+               izz="${m/12.0*(x*x+y*y)}"/>
+    </inertial>
+  </xacro:macro>
+  <!-- Cylinder inertia macro (oriented along Z before joint rotation) -->
+  <xacro:macro name="cylinder_inertia" params="m r h">
+    <inertial>
+      <mass value="${m}"/>
+      <inertia ixx="${m/12.0*(3*r*r+h*h)}" ixy="0" ixz="0"
+               iyy="${m/12.0*(3*r*r+h*h)}" iyz="0"
+               izz="${0.5*m*r*r}"/>
+    </inertial>
+  </xacro:macro>
+  <!-- Wheel macro (creates link + joint + Gazebo friction) -->
+  <xacro:macro name="mecanum_wheel" params="name x_pos y_pos fdir1_y">
+    <link name="${name}">
+      <!-- Tire -->
+      <visual>
+        <geometry><cylinder radius="${wheel_radius}" length="${wheel_width}"/></geometry>
+        <origin xyz="0 0 0" rpy="${pi/2} 0 0"/>
+        <material name="dark_rubber"/>
+      </visual>
+      <!-- Hub cap -->
+      <visual>
+        <geometry><cylinder radius="${wheel_radius*0.45}" length="${wheel_width+0.005}"/></geometry>
+        <origin xyz="0 0 0" rpy="${pi/2} 0 0"/>
+        <material name="silver"/>
+      </visual>
+      <collision>
+        <geometry><cylinder radius="${wheel_radius}" length="${wheel_width}"/></geometry>
+        <origin xyz="0 0 0" rpy="${pi/2} 0 0"/>
+      </collision>
+      <xacro:cylinder_inertia m="${wheel_mass}" r="${wheel_radius}" h="${wheel_width}"/>
+    </link>
+    <joint name="${name}_joint" type="continuous">
+      <parent link="base_link"/>
+      <child link="${name}"/>
+      <origin xyz="${x_pos} ${y_pos} -0.04" rpy="0 0 0"/>
+      <axis xyz="0 1 0"/>
+      <limit effort="10.0" velocity="10.0"/>
+      <dynamics damping="0.1" friction="0.01"/>
+    </joint>
+    <!-- Mecanum anisotropic friction -->
+    <gazebo reference="${name}">
+      <surface>
+        <friction>
+          <ode>
+            <mu>1.0</mu>
+            <mu2>0.01</mu2>
+            <fdir1>1 ${fdir1_y} 0</fdir1>
+          </ode>
+        </friction>
+        <contact>
+          <ode>
+            <soft_cfm>0</soft_cfm>
+            <soft_erp>0.2</soft_erp>
+            <kp>5000</kp>
+            <kd>2000</kd>
+            <max_vel>0.01</max_vel>
+            <min_depth>0.001</min_depth>
+          </ode>
+        </contact>
+      </surface>
+    </gazebo>
+  </xacro:macro>
+  <!-- ================================================================ -->
+  <!-- MATERIALS                                                         -->
+  <!-- ================================================================ -->
+  <material name="chassis_red">
+    <color rgba="0.75 0.12 0.12 1"/>
+  </material>
+  <material name="deck_dark">
+    <color rgba="0.18 0.18 0.20 1"/>
+  </material>
+  <material name="dark_rubber">
+    <color rgba="0.12 0.12 0.12 1"/>
+  </material>
+  <material name="silver">
+    <color rgba="0.72 0.72 0.75 1"/>
+  </material>
+  <material name="sensor_blue">
+    <color rgba="0.15 0.35 0.75 1"/>
+  </material>
+  <material name="sensor_black">
+    <color rgba="0.08 0.08 0.10 1"/>
+  </material>
+  <material name="pcb_green">
+    <color rgba="0.12 0.55 0.22 1"/>
+  </material>
+  <material name="radar_gray">
+    <color rgba="0.45 0.45 0.50 1"/>
+  </material>
+  <material name="bumper_dark">
+    <color rgba="0.20 0.20 0.22 1"/>
+  </material>
+  <material name="battery_blue">
+    <color rgba="0.10 0.20 0.50 1"/>
+  </material>
+  <material name="antenna_black">
+    <color rgba="0.05 0.05 0.08 1"/>
+  </material>
+  <material name="orange_accent">
+    <color rgba="0.95 0.55 0.05 1"/>
+  </material>
+  <!-- ================================================================ -->
+  <!-- BASE LINK (Main chassis body)                                     -->
+  <!-- ================================================================ -->
+  <link name="base_link">
+    <!-- Main chassis body -->
+    <visual>
+      <geometry><box size="${chassis_length} ${chassis_width} ${chassis_height}"/></geometry>
+      <origin xyz="0 0 0" rpy="0 0 0"/>
+      <material name="chassis_red"/>
+    </visual>
+    <!-- Chamfered front nose (angled wedge effect using a smaller box) -->
+    <visual>
+      <geometry><box size="0.06 0.24 0.06"/></geometry>
+      <origin xyz="0.26 0 -0.01" rpy="0 0.25 0"/>
+      <material name="chassis_red"/>
+    </visual>
+    <!-- Side skirt left -->
+    <visual>
+      <geometry><box size="0.44 0.015 0.05"/></geometry>
+      <origin xyz="0 0.155 -0.02" rpy="0 0 0"/>
+      <material name="bumper_dark"/>
+    </visual>
+    <!-- Side skirt right -->
+    <visual>
+      <geometry><box size="0.44 0.015 0.05"/></geometry>
+      <origin xyz="0 -0.155 -0.02" rpy="0 0 0"/>
+      <material name="bumper_dark"/>
+    </visual>
+    <collision>
+      <geometry><box size="${chassis_length} ${chassis_width} ${chassis_height}"/></geometry>
+    </collision>
+    <xacro:box_inertia m="${chassis_mass}" x="${chassis_length}" y="${chassis_width}" z="${chassis_height}"/>
+  </link>
+  <gazebo reference="base_link">
+    <surface>
+      <friction><ode><mu>0.1</mu><mu2>0.1</mu2></ode></friction>
+    </surface>
+  </gazebo>
+  <!-- ================================================================ -->
+  <!-- UPPER DECK (Electronics platform)                                 -->
+  <!-- ================================================================ -->
+  <link name="upper_deck">
+    <!-- Deck plate -->
+    <visual>
+      <geometry><box size="${upper_deck_length} ${upper_deck_width} ${upper_deck_height}"/></geometry>
+      <material name="deck_dark"/>
+    </visual>
+    <!-- Front-left standoff -->
+    <visual>
+      <geometry><cylinder radius="0.008" length="0.04"/></geometry>
+      <origin xyz="0.15 0.10 -0.02" rpy="0 0 0"/>
+      <material name="silver"/>
+    </visual>
+    <!-- Front-right standoff -->
+    <visual>
+      <geometry><cylinder radius="0.008" length="0.04"/></geometry>
+      <origin xyz="0.15 -0.10 -0.02" rpy="0 0 0"/>
+      <material name="silver"/>
+    </visual>
+    <!-- Rear-left standoff -->
+    <visual>
+      <geometry><cylinder radius="0.008" length="0.04"/></geometry>
+      <origin xyz="-0.15 0.10 -0.02" rpy="0 0 0"/>
+      <material name="silver"/>
+    </visual>
+    <!-- Rear-right standoff -->
+    <visual>
+      <geometry><cylinder radius="0.008" length="0.04"/></geometry>
+      <origin xyz="-0.15 -0.10 -0.02" rpy="0 0 0"/>
+      <material name="silver"/>
+    </visual>
+    <collision>
+      <geometry><box size="${upper_deck_length} ${upper_deck_width} ${upper_deck_height}"/></geometry>
+    </collision>
+    <xacro:box_inertia m="${upper_deck_mass}" x="${upper_deck_length}" y="${upper_deck_width}" z="${upper_deck_height}"/>
+  </link>
+  <joint name="upper_deck_joint" type="fixed">
     <parent link="base_link"/>
-    <child  link="chassis"/>
-    <origin xyz="0 0 0" rpy="0 0 0"/>
-  </joint>
-  <link name="chassis">
-    <visual name="chassis_visual">
-      <origin xyz="0 0 0" rpy="0 0 0"/>
-      <geometry>
-        <box size="${chassis_x} ${chassis_y} ${chassis_z}"/>
-      </geometry>
-      <material name="green"/>
-    </visual>
-    <collision name="chassis_collision">
-      <origin xyz="0 0 0" rpy="0 0 0"/>
-      <geometry>
-        <box size="${chassis_x} ${chassis_y} ${chassis_z}"/>
-      </geometry>
-    </collision>
-    <inertial>
-      <origin xyz="0 0 0" rpy="0 0 0"/>
-      <mass value="10.0"/>
-      <inertia ixx="0.4167" ixy="0" ixz="0"
-               iyy="1.4167" iyz="0"
-               izz="1.6667"/>
-    </inertial>
-  </link>
-  <!-- ===================== -->
-  <!-- Caster                 -->
-  <!-- ===================== -->
-  <link name="caster">
-    <visual name="caster_visual">
-      <origin xyz="0 0 0" rpy="0 0 0"/>
-      <geometry>
-        <sphere radius="0.05"/>
-      </geometry>
-      <material name="gray"/>
-    </visual>
-    <collision name="caster_collision">
-      <origin xyz="0 0 0" rpy="0 0 0"/>
-      <geometry>
-        <sphere radius="0.05"/>
-      </geometry>
-    </collision>
-  </link>
-  <joint name="joint_caster" type="fixed">
-    <parent link="chassis"/>
-    <child  link="caster"/>
-    <origin xyz="-0.15 0 -0.05" rpy="0 0 0"/>
-  </joint>
-  <!-- ===================== -->
-  <!-- Wheels (clean frames)  -->
-  <!-- ===================== -->
-  <link name="left_wheel">
-    <visual name="left_wheel_visual">
-      <!-- Cylinder is Z-axis by default; roll by pi/2 about X to align axle with Y -->
-      <origin xyz="0 0 0" rpy="${pi/2} 0 0"/>
-      <geometry>
-        <cylinder radius="${wheel_radius}" length="${wheel_width}"/>
-      </geometry>
-      <material name="gray"/>
-    </visual>
-    <collision name="left_wheel_collision">
-      <origin xyz="0 0 0" rpy="${pi/2} 0 0"/>
-      <geometry>
-        <cylinder radius="${wheel_radius}" length="${wheel_width}"/>
-      </geometry>
-    </collision>
-    <inertial>
-      <origin xyz="0 0 0" rpy="0 0 0"/>
-      <mass value="5"/>
-      <inertia ixx="1.0" ixy="0.0" ixz="0.0"
-               iyy="1.0" iyz="0.0"
-               izz="1.0"/>
-    </inertial>
-  </link>
-  <link name="right_wheel">
-    <visual name="right_wheel_visual">
-      <origin xyz="0 0 0" rpy="${pi/2} 0 0"/>
-      <geometry>
-        <cylinder radius="${wheel_radius}" length="${wheel_width}"/>
-      </geometry>
-      <material name="gray"/>
-    </visual>
-    <collision name="right_wheel_collision">
-      <origin xyz="0 0 0" rpy="${pi/2} 0 0"/>
-      <geometry>
-        <cylinder radius="${wheel_radius}" length="${wheel_width}"/>
-      </geometry>
-    </collision>
-    <inertial>
-      <origin xyz="0 0 0" rpy="0 0 0"/>
-      <mass value="5"/>
-      <inertia ixx="1.0" ixy="0.0" ixz="0.0"
-               iyy="1.0" iyz="0.0"
-               izz="1.0"/>
-    </inertial>
-  </link>
-  <!-- Wheel joints -->
-  <joint type="continuous" name="left_wheel_hinge">
-    <origin xyz="${wheel_x} ${wheel_y} 0" rpy="0 0 0"/>
+    <child link="upper_deck"/>
+    <origin xyz="-0.02 0 0.065" rpy="0 0 0"/>
+  </joint>
+  <!-- ================================================================ -->
+  <!-- FRONT BUMPER                                                      -->
+  <!-- ================================================================ -->
+  <link name="front_bumper">
+    <!-- Main bumper bar -->
+    <visual>
+      <geometry><box size="0.025 0.28 0.06"/></geometry>
+      <material name="bumper_dark"/>
+    </visual>
+    <!-- Left bumper end cap -->
+    <visual>
+      <geometry><cylinder radius="0.03" length="0.025"/></geometry>
+      <origin xyz="0 0.14 0" rpy="0 ${pi/2} 0"/>
+      <material name="bumper_dark"/>
+    </visual>
+    <!-- Right bumper end cap -->
+    <visual>
+      <geometry><cylinder radius="0.03" length="0.025"/></geometry>
+      <origin xyz="0 -0.14 0" rpy="0 ${pi/2} 0"/>
+      <material name="bumper_dark"/>
+    </visual>
+    <collision>
+      <geometry><box size="0.025 0.32 0.06"/></geometry>
+    </collision>
+    <xacro:box_inertia m="0.15" x="0.025" y="0.32" z="0.06"/>
+  </link>
+  <joint name="front_bumper_joint" type="fixed">
     <parent link="base_link"/>
-    <child  link="left_wheel"/>
-    <axis xyz="0 1 0"/>
-    <limit effort="100" velocity="100"/>
-  </joint>
-  <joint type="continuous" name="right_wheel_hinge">
-    <origin xyz="${wheel_x} ${-wheel_y} 0" rpy="0 0 0"/>
+    <child link="front_bumper"/>
+    <origin xyz="0.265 0 -0.01" rpy="0 0 0"/>
+  </joint>
+  <!-- ================================================================ -->
+  <!-- REAR BUMPER                                                       -->
+  <!-- ================================================================ -->
+  <link name="rear_bumper">
+    <visual>
+      <geometry><box size="0.02 0.26 0.05"/></geometry>
+      <material name="bumper_dark"/>
+    </visual>
+    <collision>
+      <geometry><box size="0.02 0.26 0.05"/></geometry>
+    </collision>
+    <xacro:box_inertia m="0.12" x="0.02" y="0.26" z="0.05"/>
+  </link>
+  <joint name="rear_bumper_joint" type="fixed">
     <parent link="base_link"/>
-    <child  link="right_wheel"/>
-    <axis xyz="0 1 0"/>
-    <limit effort="100" velocity="100"/>
-  </joint>
-  <!-- ===================== -->
-  <!-- Camera                 -->
-  <!-- ===================== -->
-  <link name="camera">
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